File: 1sqinch555.sch (KiCad schematic (older format))
At the start: 68 parts, among them J1 Conn_01x01, J10 Conn_01x01, J11 Conn_01x01, J12 Conn_01x01, J13 Conn_01x01, J14 Conn_01x01, J15 Conn_01x01, J16 Conn_01x01, J17 Conn_01x01, J18 Conn_01x01, J19 Conn_01x01, J2 Conn_01x01, J20 Conn_01x01, J21 Conn_01x01, J22 Conn_01x01, J23 Conn_01x01, J24 Conn_01x01, J25 Conn_01x01, J26 Conn_01x01, J27 Conn_01x01, J28 Conn_01x01, J29 Conn_01x01, J3 Conn_01x01, J30 Conn_01x01, J31 Conn_01x01, J32 Conn_01x01, J33 Conn_01x01, J34 Conn_01x01, J35 Conn_01x01, J4 Conn_01x01, J5 Conn_01x01, J6 Conn_01x01, J7 Conn_01x01, J8 Conn_01x01, J9 Conn_01x01, U1 LM555, U2 4020

Commit message: changed 0603 to 0805
Parts:
- added R10, R2, R3, R4, R5, R6, R7, R8, R9: 300, 1sqinch555_fp:R_0805, symbol 1sqinch:R
- C1, C2: footprint 1sqinch555_fp:C_0603 -> 1sqinch555_fp:C_0805
- D1, D10, D11, D12, D13, D14, D15, D16, D17, D18, D19, D2, D20, D21, D22, D23, D24, D25, D26, D27, D3, D4, D5, D6, D7, D8, D9: footprint 1sqinch555_fp:D_0603 -> 1sqinch555_fp:LED-0805
- R1: footprint 1sqinch555_fp:R_0603 -> 1sqinch555_fp:R_0805
Connections:
- wire segments 125 -> 134

Commit message: mods
Other:
- note added: "Vf = 2.1 V\nIf = 10mA\nRled = 9 - (2.1*3) V / 10mA\nRled = 270 ohms"
Changed lines of the file:
@@
 	9625 4900 10100 4900
 Connection ~ 10100 4900
+Text Notes 6975 6500 0    50   ~ 0
+Vf = 2.1 V\nIf = 10mA\nRled = 9 - (2.1*3) V / 10mA\nRled = 270 ohms
 $EndSCHEMATC
